File: First_keyboard30/First_keyboard30.sch (KiCad schematic (older format))
At the start: 70 parts, among them SW1 RESET_SW, SW10 RESET_SW, SW11 RESET_SW, SW12 RESET_SW, SW13 RESET_SW, SW14 RESET_SW, SW15 RESET_SW, SW16 RESET_SW, SW17 RESET_SW, SW18 RESET_SW, SW19 RESET_SW, SW2 RESET_SW, SW20 RESET_SW, SW21 RESET_SW, SW22 RESET_SW, SW23 RESET_SW, SW24 RESET_SW, SW25 RESET_SW, SW26 RESET_SW, SW27 RESET_SW, SW28 RESET_SW, SW29 RESET_SW, SW3 RESET_SW, SW30 RESET_SW, SW31 RESET_SW, SW32 RESET_SW, SW33 RESET_SW, SW34 RESET_SW, SW35 RESET_SW, SW4 RESET_SW, SW5 RESET_SW, SW6 RESET_SW, SW7 RESET_SW, SW8 RESET_SW, SW9 RESET_SW, U1 ProMicro

Commit message: pcb update
Parts:
- D1, D10, D11, D12, D13, D14, D15, D16, D17, D18, D19, D2, D20, D21, D22, D23, D24, D25, D26, D27, D28, D29, D3, D30, D31, D32, D33, D34, D4, D5, D6, D7, D8, D9: footprint (none) -> kbd:D3_TH_SMD
- SW1: footprint (none) -> kbd:ResetSW
- SW10, SW11, SW12, SW13, SW14, SW15, SW16, SW17, SW18, SW19, SW2, SW20, SW21, SW22, SW23, SW24, SW25, SW26, SW27, SW28, SW29, SW3, SW30, SW32, SW33, SW34, SW4, SW5, SW6, SW7, SW8, SW9: value RESET_SW -> KEY_SW; footprint (none) -> kbd:CherryMX_1u
- SW31, SW35: value RESET_SW -> KEY_SW; footprint (none) -> Keebio-Parts:MX-Alps-Choc-2U
- U1: footprint (none) -> Keebio-Parts:ArduinoProMicro

Commit message: rename
Other:
- note added: "первый\n"
- note removed: "First\n"
Changed lines of the file:
@@
 	0    1    1    0
 $EndComp
-Text Notes 9760 7080 2    394  Italic 79
-First\n
+Text Notes 10110 7040 2    394  Italic 79
+первый\n
 Text GLabel 5000 1400 1    50   Input ~ 0
 col0
