File: VTOROY/VTOROY.sch (KiCad schematic (older format))
At the start: 2 parts

Commit message: save
Parts:
- removed D?: DIODE, symbol Simulation_SPICE:DIODE
- added D1, D10, D11, D12, D13, D14, D15, D16, D17, D18, D19, D2, D20, D21, D22, D23, D24, D25, D26, D27, D28, D29, D3, D30, D31, D32, D33, D4, D5, D6, D7, D8, D9: DIODE, kbd:D3_TH_SMD, symbol Simulation_SPICE:DIODE
- added J1: MJ-4PP-9, kbd:MJ-4PP-9_1side, symbol kbd:MJ-4PP-9
- added SW1: RESET_SW, kbd:ResetSW, symbol kbd:SW_PUSH
- added SW10, SW11, SW12, SW13, SW14, SW15, SW16, SW17, SW18, SW19, SW2, SW20, SW21, SW22, SW23, SW24, SW25, SW26, SW27, SW28, SW29, SW3, SW30, SW31, SW32, SW33, SW34, SW4, SW5, SW6, SW7, SW8, SW9: SW_PUSH, keyswitches:SW_MX_reversible, symbol kbd:SW_PUSH
- added U2: ProMicro, kbd:ProMicro_v3, symbol kbd:ProMicro
- U1: renamed from U?; footprint (none) -> kbd:ProMicro_v3
Connections:
- net labels added: GND, VCC, col0, col1, col2, col3, col4, col5, col6, data, reset, row0, row1, row2, row3, row4
- wire segments 0 -> 81
- no-connect marks 0 -> 13
Other:
- note added: "7x5 col row\n"
- note added: "trrs jack"
- moved on the sheet: U1
