File: tron_clone/tron_clone.sch (KiCad schematic (older format))
At the start: 65 parts

Commit message: new keyboard
Parts:
- D? (x31): symbol Simulation_SPICE:DIODE -> tron_clone-rescue:DIODE-Simulation_SPICE
Changed lines of the file:
@@
 $EndComp
 $Comp
-L Simulation_SPICE:DIODE D?
+L tron_clone-rescue:DIODE-Simulation_SPICE D?
 U 1 1 5EFF9967
 P 10600 2300
@@
 $EndComp
 $Comp
-L Simulation_SPICE:DIODE D?
+L tron_clone-rescue:DIODE-Simulation_SPICE D?
 U 1 1 5EFF0D75
 P 10600 1650
@@
 $EndComp
 $Comp
-L Simulation_SPICE:DIODE D?
+L tron_clone-rescue:DIODE-Simulation_SPICE D?
 U 1 1 5EFF0D67
 P 10600 2950
@@
 $EndComp
 $Comp
-L Simulation_SPICE:DIODE D?
+L tron_clone-rescue:DIODE-Simulation_SPICE D?
 U 1 1 5EFF0D59
 P 7600 4300
@@
 $EndComp
 $Comp
-L Simulation_SPICE:DIODE D?
+L tron_clone-rescue:DIODE-Simulation_SPICE D?
 U 1 1 5EFF0D4B
 P 6605 4300
@@
 $EndComp
 $Comp
-L Simulation_SPICE:DIODE D?
+L tron_clone-rescue:DIODE-Simulation_SPICE D?
 U 1 1 5EFF0D3D
 P 5600 4300
@@
 $EndComp
 $Comp
-L Simulation_SPICE:DIODE D?
+L tron_clone-rescue:DIODE-Simulation_SPICE D?
 U 1 1 5EFF0D2F
 P 4600 4300
@@
 $EndComp
 $Comp
-L Simulation_SPICE:DIODE D?
+L tron_clone-rescue:DIODE-Simulation_SPICE D?
 U 1 1 5EFE891B
 P 8605 2950
@@
 $EndComp
 $Comp
-L Simulation_SPICE:DIODE D?
+L tron_clone-rescue:DIODE-Simulation_SPICE D?
 U 1 1 5EFE890D
 P 7600 2950
@@
 $EndComp
 $Comp
-L Simulation_SPICE:DIODE D?
+L tron_clone-rescue:DIODE-Simulation_SPICE D?
 U 1 1 5EFE88FF
 P 6605 2950
@@
 $EndComp
 $Comp
-L Simulation_SPICE:DIODE D?
+L tron_clone-rescue:DIODE-Simulation_SPICE D?
 U 1 1 5EFE88F1
 P 5600 2950
@@
 $EndComp
 $Comp
-L Simulation_SPICE:DIODE D?
+L tron_clone-rescue:DIODE-Simulation_SPICE D?
 U 1 1 5EFE88E3
 P 4600 2950
@@
 $EndComp
 $Comp
-L Simulation_SPICE:DIODE D?
+L tron_clone-rescue:DIODE-Simulation_SPICE D?
 U 1 1 5EFDC36D
 P 9600 2300
@@
 $EndComp
 $Comp
-L Simulation_SPICE:DIODE D?
+L tron_clone-rescue:DIODE-Simulation_SPICE D?
 U 1 1 5EFDC35F
 P 8605 2300
@@
 $EndComp
 $Comp
-L Simulation_SPICE:DIODE D?
+L tron_clone-rescue:DIODE-Simulation_SPICE D?
 U 1 1 5EFDC351
 P 7600 2300
@@
 $EndComp
 $Comp
-L Simulation_SPICE:DIODE D?
+L tron_clone-rescue:DIODE-Simulation_SPICE D?
 U 1 1 5EFDC343
 P 6605 2300
@@
 $EndComp
 $Comp
-L Simulation_SPICE:DIODE D?
+L tron_clone-rescue:DIODE-Simulation_SPICE D?
 U 1 1 5EFDC335
 P 5600 2300
@@
 $EndComp
 $Comp
-L Simulation_SPICE:DIODE D?
+L tron_clone-rescue:DIODE-Simulation_SPICE D?
 U 1 1 5EFDC327
 P 4600 2300
@@
 $EndComp
 $Comp
-L Simulation_SPICE:DIODE D?
+L tron_clone-rescue:DIODE-Simulation_SPICE D?
 U 1 1 5EFC8DDB
 P 9600 1650
@@
 $EndComp
 $Comp
-L Simulation_SPICE:DIODE D?
+L tron_clone-rescue:DIODE-Simulation_SPICE D?
 U 1 1 5EFC74B5
 P 8605 1650
@@
 $EndComp
 $Comp
-L Simulation_SPICE:DIODE D?
+L tron_clone-rescue:DIODE-Simulation_SPICE D?
 U 1 1 5EFC6B5B
 P 7600 1650
@@
 $EndComp
 $Comp
-L Simulation_SPICE:DIODE D?
+L tron_clone-rescue:DIODE-Simulation_SPICE D?
 U 1 1 5EFC5D99
 P 6605 1650
@@
 $EndComp
 $Comp
-L Simulation_SPICE:DIODE D?
+L tron_clone-rescue:DIODE-Simulation_SPICE D?
 U 1 1 5EFC388B
 P 5600 1650
@@
 $EndComp
 $Comp
-L Simulation_SPICE:DIODE D?
+L tron_clone-rescue:DIODE-Simulation_SPICE D?
 U 1 1 5EFBC4C1
 P 4600 1650
@@
 $EndComp
 $Comp
-L Simulation_SPICE:DIODE D?
+L tron_clone-rescue:DIODE-Simulation_SPICE D?
 U 1 1 5EFF992F
 P 5595 3650
@@
 $EndComp
 $Comp
-L Simulation_SPICE:DIODE D?
+L tron_clone-rescue:DIODE-Simulation_SPICE D?
 U 1 1 5EFF993D
 P 6600 3650
@@
 $EndComp
 $Comp
-L Simulation_SPICE:DIODE D?
+L tron_clone-rescue:DIODE-Simulation_SPICE D?
 U 1 1 5EFF994B
 P 7595 3650
@@
 $EndComp
 $Comp
-L Simulation_SPICE:DIODE D?
+L tron_clone-rescue:DIODE-Simulation_SPICE D?
 U 1 1 5EFF9959
 P 8605 3650
@@
 $EndComp
 $Comp
-L Simulation_SPICE:DIODE D?
+L tron_clone-rescue:DIODE-Simulation_SPICE D?
 U 1 1 5F002211
 P 9605 3650
@@
 $EndComp
 $Comp
-L Simulation_SPICE:DIODE D?
+L tron_clone-rescue:DIODE-Simulation_SPICE D?
 U 1 1 5F166C86
 P 9600 2950
@@
 $EndComp
 $Comp
-L Simulation_SPICE:DIODE D?
+L tron_clone-rescue:DIODE-Simulation_SPICE D?
 U 1 1 5F1674AD
 P 4600 3650
