File: 42Key/42Key.sch (KiCad schematic (older format))
At the start: 45 parts, among them SW0 RESET_SW

Commit message: save
Parts:
- D1, D10, D11, D12, D13, D14, D15, D16, D17, D18, D19, D2, D20, D21, D3, D4, D5, D6, D7, D8, D9: renamed from D?; footprint (none) -> kbd:D3_TH_SMD; symbol Simulation_SPICE:DIODE -> 42Key-rescue:DIODE-Simulation_SPICE
- J1: renamed from J?; footprint (none) -> kbd:MJ-4PP-9
- SW0: footprint (none) -> kbd:ResetSW
- gave numbers to parts that had none: 22
Connections:
- wire segments 54 -> 56

Commit message: compleate
Parts:
- SW1, SW10, SW11, SW12, SW13, SW14, SW15, SW16, SW17, SW18, SW2, SW3, SW4, SW5, SW6, SW7, SW8, SW9: footprint (none) -> Keebio-Parts:Triple-Dual-1u-LED
- SW19, SW20, SW21: footprint (none) -> Keebio-Parts:Triple-Dual-2u-LED
- U1: footprint (none) -> kbd:ProMicro_v2
Changed lines of the file:
@@
 F 0 "U1" H 2000 3387 60  0000 C CNN
 F 1 "ProMicro" H 2000 3281 60  0000 C CNN
-F 2 "" H 2100 1300 60  0001 C CNN
+F 2 "kbd:ProMicro_v2" H 2100 1300 60  0001 C CNN
 F 3 "" H 2100 1300 60  0000 C CNN
 	1    2000 2350
@@
 F 0 "SW1" H 4300 1755 50  0000 C CNN
 F 1 "SW_PUSH" H 4300 1664 50  0000 C CNN
-F 2 "" H 4300 1500 50  0001 C CNN
+F 2 "Keebio-Parts:Triple-Dual-1u-LED" H 4300 1500 50  0001 C CNN
 F 3 "" H 4300 1500 50  0000 C CNN
 	1    4300 1500
@@
 F 0 "SW4" H 5300 1755 50  0000 C CNN
 F 1 "SW_PUSH" H 5300 1664 50  0000 C CNN
-F 2 "" H 5300 1500 50  0001 C CNN
+F 2 "Keebio-Parts:Triple-Dual-1u-LED" H 5300 1500 50  0001 C CNN
 F 3 "" H 5300 1500 50  0000 C CNN
 	1    5300 1500
@@
 F 0 "SW7" H 6300 1755 50  0000 C CNN
 F 1 "SW_PUSH" H 6300 1664 50  0000 C CNN
-F 2 "" H 6300 1500 50  0001 C CNN
+F 2 "Keebio-Parts:Triple-Dual-1u-LED" H 6300 1500 50  0001 C CNN
 F 3 "" H 6300 1500 50  0000 C CNN
 	1    6300 1500
@@
 F 0 "SW11" H 7300 1755 50  0000 C CNN
 F 1 "SW_PUSH" H 7300 1664 50  0000 C CNN
-F 2 "" H 7300 1500 50  0001 C CNN
+F 2 "Keebio-Parts:Triple-Dual-1u-LED" H 7300 1500 50  0001 C CNN
 F 3 "" H 7300 1500 50  0000 C CNN
 	1    7300 1500
@@
 F 0 "SW15" H 8300 1755 50  0000 C CNN
 F 1 "SW_PUSH" H 8300 1664 50  0000 C CNN
-F 2 "" H 8300 1500 50  0001 C CNN
+F 2 "Keebio-Parts:Triple-Dual-1u-LED" H 8300 1500 50  0001 C CNN
 F 3 "" H 8300 1500 50  0000 C CNN
 	1    8300 1500
@@
 F 0 "SW18" H 9300 1755 50  0000 C CNN
 F 1 "SW_PUSH" H 9300 1664 50  0000 C CNN
-F 2 "" H 9300 1500 50  0001 C CNN
+F 2 "Keebio-Parts:Triple-Dual-1u-LED" H 9300 1500 50  0001 C CNN
 F 3 "" H 9300 1500 50  0000 C CNN
 	1    9300 1500
@@
 F 0 "SW2" H 4300 2255 50  0000 C CNN
 F 1 "SW_PUSH" H 4300 2164 50  0000 C CNN
-F 2 "" H 4300 2000 50  0001 C CNN
+F 2 "Keebio-Parts:Triple-Dual-1u-LED" H 4300 2000 50  0001 C CNN
 F 3 "" H 4300 2000 50  0000 C CNN
 	1    4300 2000
@@
 F 0 "SW5" H 5300 2255 50  0000 C CNN
 F 1 "SW_PUSH" H 5300 2164 50  0000 C CNN
-F 2 "" H 5300 2000 50  0001 C CNN
+F 2 "Keebio-Parts:Triple-Dual-1u-LED" H 5300 2000 50  0001 C CNN
 F 3 "" H 5300 2000 50  0000 C CNN
 	1    5300 2000
@@
 F 0 "SW8" H 6300 2255 50  0000 C CNN
 F 1 "SW_PUSH" H 6300 2164 50  0000 C CNN
-F 2 "" H 6300 2000 50  0001 C CNN
+F 2 "Keebio-Parts:Triple-Dual-1u-LED" H 6300 2000 50  0001 C CNN
 F 3 "" H 6300 2000 50  0000 C CNN
 	1    6300 2000
@@
 F 0 "SW12" H 7300 2255 50  0000 C CNN
 F 1 "SW_PUSH" H 7300 2164 50  0000 C CNN
-F 2 "" H 7300 2000 50  0001 C CNN
+F 2 "Keebio-Parts:Triple-Dual-1u-LED" H 7300 2000 50  0001 C CNN
 F 3 "" H 7300 2000 50  0000 C CNN
 	1    7300 2000
@@
 F 0 "SW16" H 8300 2255 50  0000 C CNN
 F 1 "SW_PUSH" H 8300 2164 50  0000 C CNN
-F 2 "" H 8300 2000 50  0001 C CNN
+F 2 "Keebio-Parts:Triple-Dual-1u-LED" H 8300 2000 50  0001 C CNN
 F 3 "" H 8300 2000 50  0000 C CNN
 	1    8300 2000
@@
 F 0 "SW19" H 9300 2255 50  0000 C CNN
 F 1 "SW_PUSH" H 9300 2164 50  0000 C CNN
-F 2 "" H 9300 2000 50  0001 C CNN
+F 2 "Keebio-Parts:Triple-Dual-2u-LED" H 9300 2000 50  0001 C CNN
 F 3 "" H 9300 2000 50  0000 C CNN
 	1    9300 2000
@@
 F 0 "SW3" H 4300 2755 50  0000 C CNN
 F 1 "SW_PUSH" H 4300 2664 50  0000 C CNN
-F 2 "" H 4300 2500 50  0001 C CNN
+F 2 "Keebio-Parts:Triple-Dual-1u-LED" H 4300 2500 50  0001 C CNN
 F 3 "" H 4300 2500 50  0000 C CNN
 	1    4300 2500
@@
 F 0 "SW6" H 5300 2755 50  0000 C CNN
 F 1 "SW_PUSH" H 5300 2664 50  0000 C CNN
-F 2 "" H 5300 2500 50  0001 C CNN
+F 2 "Keebio-Parts:Triple-Dual-1u-LED" H 5300 2500 50  0001 C CNN
 F 3 "" H 5300 2500 50  0000 C CNN
 	1    5300 2500
@@
 F 0 "SW9" H 6300 2755 50  0000 C CNN
 F 1 "SW_PUSH" H 6300 2664 50  0000 C CNN
-F 2 "" H 6300 2500 50  0001 C CNN
+F 2 "Keebio-Parts:Triple-Dual-1u-LED" H 6300 2500 50  0001 C CNN
 F 3 "" H 6300 2500 50  0000 C CNN
 	1    6300 2500
@@
 F 0 "SW13" H 7300 2755 50  0000 C CNN
 F 1 "SW_PUSH" H 7300 2664 50  0000 C CNN
-F 2 "" H 7300 2500 50  0001 C CNN
+F 2 "Keebio-Parts:Triple-Dual-1u-LED" H 7300 2500 50  0001 C CNN
 F 3 "" H 7300 2500 50  0000 C CNN
 	1    7300 2500
@@
 F 0 "SW17" H 8300 2755 50  0000 C CNN
 F 1 "SW_PUSH" H 8300 2664 50  0000 C CNN
-F 2 "" H 8300 2500 50  0001 C CNN
+F 2 "Keebio-Parts:Triple-Dual-1u-LED" H 8300 2500 50  0001 C CNN
 F 3 "" H 8300 2500 50  0000 C CNN
 	1    8300 2500
@@
 F 0 "SW20" H 9300 2755 50  0000 C CNN
 F 1 "SW_PUSH" H 9300 2664 50  0000 C CNN
-F 2 "" H 9300 2500 50  0001 C CNN
+F 2 "Keebio-Parts:Triple-Dual-2u-LED" H 9300 2500 50  0001 C CNN
 F 3 "" H 9300 2500 50  0000 C CNN
 	1    9300 2500
@@
 F 0 "SW10" H 6300 3255 50  0000 C CNN
 F 1 "SW_PUSH" H 6300 3164 50  0000 C CNN
-F 2 "" H 6300 3000 50  0001 C CNN
+F 2 "Keebio-Parts:Triple-Dual-1u-LED" H 6300 3000 50  0001 C CNN
 F 3 "" H 6300 3000 50  0000 C CNN
 	1    6300 3000
@@
 F 0 "SW14" H 7300 3255 50  0000 C CNN
 F 1 "SW_PUSH" H 7300 3164 50  0000 C CNN
-F 2 "" H 7300 3000 50  0001 C CNN
+F 2 "Keebio-Parts:Triple-Dual-1u-LED" H 7300 3000 50  0001 C CNN
 F 3 "" H 7300 3000 50  0000 C CNN
 	1    7300 3000
@@
 F 0 "SW21" H 9300 3255 50  0000 C CNN
 F 1 "SW_PUSH" H 9300 3164 50  0000 C CNN
-F 2 "" H 9300 3000 50  0001 C CNN
+F 2 "Keebio-Parts:Triple-Dual-2u-LED" H 9300 3000 50  0001 C CNN
 F 3 "" H 9300 3000 50  0000 C CNN
 	1    9300 3000
