File: Маленький/Маленький.kicad_pcb (KiCad board)
At the start: 2 copper layers, 77.8 x 80.9 mm, 20 parts, among them SW1 SW_PUSH, SW2 SW_PUSH, SW3 SW_PUSH, SW4 SW_PUSH, SW5 SW_PUSH, U1 ProMicro

Commit message: aouto save
Parts:
- added REF**: MountingHole_2.2mm_M2, MountingHole:MountingHole_2.2mm_M2, F.Cu at (138.0, 131.4)
- added REF**: MountingHole_2.2mm_M2, MountingHole:MountingHole_2.2mm_M2, F.Cu at (177.7, 131.7)
- added REF**: MountingHole_2.2mm_M2, MountingHole:MountingHole_2.2mm_M2, F.Cu at (177.7, 90.5)
- added REF**: MountingHole_2.2mm_M2, MountingHole:MountingHole_2.2mm_M2, F.Cu at (138.0, 90.3)
Routing:
- net (no net): track 242.4 -> 244.1 mm
- net row1: track 32.4 -> 33.5 mm
- net row0: track 31.4 -> 32.0 mm
Other:
- board size 77.8 x 80.9 mm -> 77.8 x 81 mm
